File: hardware/Orbitpad_PCB.kicad_pcb (KiCad board)
At the start: 2 copper layers, 84.5 x 99.3 mm, 50 parts, among them J1 Conn_01x04_Pin, SW1 SW_Push, SW10 SW_Push, SW11 SW_Push, SW12 SW_Push, SW13 SW_Push, SW14 SW_Push, SW15 SW_Push, SW16 SW_Push, SW2 SW_Push, SW3 SW_Push, SW4 SW_Push, SW5 SW_Push, SW6 SW_Push, SW7 SW_Push, SW8 SW_Push, SW9 SW_Push, U1 XIAO-RP2040-DIP

Commit message: Final KiCAD PCB design
These are the final Kicad files for the PCB
Parts:
- D1, D10, D11, D12, D13, D14, D15, D16, D2, D3, D4, D5, D6, D7, D8, D9: value SK6812MINI -> SK6812MINI-E; footprint LED_SMD:LED_SK6812MINI_PLCC4_3.5x3.5mm_P1.75mm -> PCM_marbastlib-various:LED_6028R; moved to B.Cu
- moved D4 66.5 mm to (114.0, 82.6), turned to 180 degrees
- moved D16 66.5 mm to (114.0, 139.5), turned to 180 degrees
- moved D12 66.4 mm to (114.0, 120.5), turned to 180 degrees
- moved D8 66.4 mm to (114.0, 101.5), turned to 180 degrees
- moved D13 48.0 mm to (171.5, 139.7), turned to 180 degrees
- moved D1 47.7 mm to (171.0, 82.5), turned to 180 degrees
- moved D5 47.6 mm to (171.0, 101.5), turned to 180 degrees
- moved D9 47.6 mm to (171.0, 120.5), turned to 180 degrees
- moved D11 28.5 mm to (133.0, 120.5), turned to 180 degrees
- moved D15 28.5 mm to (133.0, 139.5), turned to 180 degrees
- moved D3 28.5 mm to (132.9, 82.5), turned to 180 degrees
- moved D7 28.4 mm to (133.0, 101.5), turned to 180 degrees
- moved D6 9.66 mm to (152.0, 101.5), turned to 180 degrees
- moved D2 9.65 mm to (152.0, 82.5), turned to 180 degrees
- moved D14 9.55 mm to (152.0, 139.5), turned to 180 degrees
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Connections:
- D1 pad 1: Net-(D1-DOUT) -> +5V
- D1 pad 2: GND -> Net-(D1-DOUT)
- D1 pad 4: +5V -> GND
- D10 pad 1: Net-(D10-DOUT) -> +5V
- D10 pad 2: GND -> Net-(D10-DOUT)
- D10 pad 3: Net-(D10-DIN) -> Net-(D10-VSS)
- D10 pad 4: +5V -> GND
- D11 pad 1: Net-(D11-DOUT) -> +5V
- D11 pad 2: GND -> Net-(D11-DOUT)
- D11 pad 4: +5V -> GND
- D12 pad 1: Net-(D12-DOUT) -> +5V
- D12 pad 2: GND -> Net-(D12-DOUT)
- D12 pad 4: +5V -> GND
- D13 pad 1: Net-(D13-DOUT) -> +5V
- D13 pad 2: GND -> Net-(D13-DOUT)
- D13 pad 4: +5V -> GND
- D14 pad 1: Net-(D14-DOUT) -> +5V
- D14 pad 2: GND -> Net-(D14-DOUT)
- D14 pad 4: +5V -> GND
- D15 pad 1: Net-(D15-DOUT) -> +5V
- D15 pad 2: GND -> Net-(D15-DOUT)
- D15 pad 4: +5V -> GND
- D16 pad 1: unconnected-(D16-DOUT-Pad1) -> +5V
- D16 pad 2: GND -> unconnected-(D16-DOUT-Pad2)
- D16 pad 4: +5V -> GND
- D2 pad 1: Net-(D2-DOUT) -> +5V
- D2 pad 2: GND -> Net-(D2-DOUT)
- D2 pad 4: +5V -> GND
- D3 pad 1: Net-(D3-DOUT) -> +5V
- D3 pad 2: GND -> Net-(D3-DOUT)
- D3 pad 4: +5V -> GND
- D4 pad 1: Net-(D4-DOUT) -> +5V
- D4 pad 2: GND -> Net-(D4-DOUT)
- D4 pad 4: +5V -> GND
- D5 pad 1: Net-(D5-DOUT) -> +5V
- D5 pad 2: GND -> Net-(D5-DOUT)
- D5 pad 4: +5V -> GND
- D6 pad 1: Net-(D6-DOUT) -> +5V
- D6 pad 2: GND -> Net-(D6-DOUT)
- D6 pad 4: +5V -> GND
- D7 pad 1: Net-(D7-DOUT) -> +5V
- D7 pad 2: GND -> Net-(D7-DOUT)
- D7 pad 4: +5V -> GND
- D8 pad 1: Net-(D8-DOUT) -> +5V
- D8 pad 2: GND -> Net-(D8-DOUT)
- D8 pad 4: +5V -> GND
- D9 pad 1: Net-(D10-DIN) -> +5V
- D9 pad 2: GND -> Net-(D10-VSS)
- D9 pad 4: +5V -> GND
Routing:
- net /Column 3: track 501.1 -> 138.4 mm
- net /Column 2: track 374.0 -> 123.9 mm
- net /Column 1: track 246.8 -> 108.3 mm
- net /Column 0: track 184.1 -> 90.9 mm
- net +5V: track 341.7 -> 412.2 mm
- net /LED: track 21.3 -> 78.4 mm
- net /Row 0: track 64.6 -> 110.4 mm
- net GND: track 383.4 -> 426.7 mm
- net Net-(D10-DIN): track 22.7 -> 0.00 mm
- net Net-(D10-VSS): track 0.00 -> 14.2 mm
- net Net-(D2-DOUT): track 22.9 -> 14.3 mm
- net Net-(D3-DOUT): track 22.5 -> 14.1 mm
- net Net-(D5-DOUT): track 22.2 -> 14.2 mm
- net Net-(D15-DOUT): track 22.2 -> 14.2 mm
- net Net-(D14-DOUT): track 22.2 -> 14.2 mm
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Other:
- board text added: "OLED SCREEN HERE"
- board text added: "OrbitPad"
- board text added: "XIAO HERE!"
